File: KiCAD/PrawnBlaster.sch (KiCad schematic (older format))
At the start: 15 parts, among them J1 DB9_Female, J11 Flag_12, J2 Flag_15, J5 Flag_14, J8 Flag_13

Commit message: added external trigger
Parts:
- removed J1: DB9_Female, Connector_Dsub:DSUB-9_Female_Vertical_P2.77x2.84mm, symbol Connector:DB9_Female
- added J1: Conn_Coaxial, symbol Connector:Conn_Coaxial
- added U3: Pico, RPi_Pico:RPi_Pico_SMD_TH, symbol MCU_RaspberryPi_and_Boards:Pico
- added U4: SN74LV1T34DBV, Package_TO_SOT_SMD:SOT-23-5, symbol Logic_LevelTranslator:SN74LV1T34DBV
Connections:
- wire segments 49 -> 46
- no-connect marks 0 -> 36
Changed lines of the file:
@@
-$EndComp
-$Comp
-L power:GND #PWR01
-U 1 1 58133322
-P 1500 4200
-F 0 "#PWR01" H 1500 3950 50  0001 C CNN
-F 1 "GND" H 1500 4050 50  0000 C CNN
-F 2 "" H 1500 4200 50  0000 C CNN
-F 3 "" H 1500 4200 50  0000 C CNN
-	1    1500 4200
-	1    0    0    -1
 $EndComp
 $Comp
@@
 	1700 800  3100 800
 Wire Wire Line
-	3100 800  3100 2300
-Wire Wire Line
 	3100 2300 3700 2300
 Wire Wire Line
@@
 Text Notes 6650 2100 0    60   ~ 0
 Use at least 250 mW resistors!\n(70 mA @ 50 Ω)
-$Comp
-L Mechanical:MountingHole H1
-U 1 1 5FEDAB5A
-P 950 5750
-F 0 "H1" H 1050 5795 50  0000 L CNN
-F 1 "MountingHole" H 1050 5706 50  0000 L CNN
-F 2 "MountingHole:MountingHole_2.7mm_M2.5_DIN965" H 950 5750 50  0001 C CNN
-F 3 "~" H 950 5750 50  0001 C CNN
-	1    950  5750
-	1    0    0    -1
-$EndComp
-$Comp
-L Mechanical:MountingHole H2
-U 1 1 5FEDBA18
-P 950 6050
-F 0 "H2" H 1050 6095 50  0000 L CNN
-F 1 "MountingHole" H 1050 6006 50  0000 L CNN
-F 2 "MountingHole:MountingHole_2.7mm_M2.5_DIN965" H 950 6050 50  0001 C CNN
-F 3 "~" H 950 6050 50  0001 C CNN
-	1    950  6050
-	1    0    0    -1
-$EndComp
-$Comp
-L Mechanical:MountingHole H3
-U 1 1 5FEDC6AA
-P 950 6350
-F 0 "H3" H 1050 6395 50  0000 L CNN
-F 1 "MountingHole" H 1050 6306 50  0000 L CNN
-F 2 "MountingHole:MountingHole_2.7mm_M2.5_DIN965" H 950 6350 50  0001 C CNN
-F 3 "~" H 950 6350 50  0001 C CNN
-	1    950  6350
-	1    0    0    -1
-$EndComp
-$Comp
-L Mechanical:MountingHole H4
-U 1 1 5FEDD2EF
-P 950 6650
-F 0 "H4" H 1050 6695 50  0000 L CNN
-F 1 "MountingHole" H 1050 6606 50  0000 L CNN
-F 2 "MountingHole:MountingHole_2.7mm_M2.5_DIN965" H 950 6650 50  0001 C CNN
-F 3 "~" H 950 6650 50  0001 C CNN
-	1    950  6650
-	1    0    0    -1
-$EndComp
 Wire Wire Line
 	10000 2950 10200 2950
@@
 	0    -1   -1   0
 $EndComp
+Wire Wire Line
+	5100 3300 5650 3300
+Wire Wire Line
+	5650 3300 5650 2350
+Wire Wire Line
+	5650 2350 7200 2350
+Wire Wire Line
+	5100 3400 5800 3400
+Wire Wire Line
+	5800 3400 5800 2550
+Wire Wire Line
+	5800 2550 7200 2550
+Wire Wire Line
+	5100 3500 5950 3500
+Wire Wire Line
+	5950 3500 5950 2750
+Wire Wire Line
+	5950 2750 7200 2750
+Wire Wire Line
+	5100 3600 6100 3600
+Wire Wire Line
+	6100 3600 6100 2950
+Wire Wire Line
+	6100 2950 7200 2950
 $Sheet
 S 3700 2200 1400 1950
@@
 F10 "B3" O R 5100 3300 50
 $EndSheet
-Wire Wire Line
-	5100 3300 5650 3300
-Wire Wire Line
-	5650 3300 5650 2350
-Wire Wire Line
-	5650 2350 7200 2350
-Wire Wire Line
-	5100 3400 5800 3400
-Wire Wire Line
-	5800 3400 5800 2550
-Wire Wire Line
-	5800 2550 7200 2550
-Wire Wire Line
-	5100 3500 5950 3500
-Wire Wire Line
-	5950 3500 5950 2750
-Wire Wire Line
-	5950 2750 7200 2750
-Wire Wire Line
-	5100 3600 6100 3600
-Wire Wire Line
-	6100 3600 6100 2950
-Wire Wire Line
-	6100 2950 7200 2950
-$Comp
-L Connector:DB9_Female J1
-U 1 1 6148E628
-P 1100 3600
-F 0 "J1" H 1018 2908 50  0000 C CNN
-F 1 "DB9_Female" H 1018 2999 50  0000 C CNN
-F 2 "Connector_Dsub:DSUB-9_Female_Vertical_P2.77x2.84mm" H 1100 3600 50  0001 C CNN
-F 3 " ~" H 1100 3600 50  0001 C CNN
-	1    1100 3600
+$Comp
+L Mechanical:MountingHole H4
+U 1 1 5FEDD2EF
+P 950 6650
+F 0 "H4" H 1050 6695 50  0000 L CNN
+F 1 "MountingHole" H 1050 6606 50  0000 L CNN
+F 2 "MountingHole:MountingHole_2.7mm_M2.5_DIN965" H 950 6650 50  0001 C CNN
+F 3 "~" H 950 6650 50  0001 C CNN
+	1    950  6650
+	1    0    0    -1
+$EndComp
+$Comp
+L Mechanical:MountingHole H3
+U 1 1 5FEDC6AA
+P 950 6350
+F 0 "H3" H 1050 6395 50  0000 L CNN
+F 1 "MountingHole" H 1050 6306 50  0000 L CNN
+F 2 "MountingHole:MountingHole_2.7mm_M2.5_DIN965" H 950 6350 50  0001 C CNN
+F 3 "~" H 950 6350 50  0001 C CNN
+	1    950  6350
+	1    0    0    -1
+$EndComp
+$Comp
+L Mechanical:MountingHole H2
+U 1 1 5FEDBA18
+P 950 6050
+F 0 "H2" H 1050 6095 50  0000 L CNN
+F 1 "MountingHole" H 1050 6006 50  0000 L CNN
+F 2 "MountingHole:MountingHole_2.7mm_M2.5_DIN965" H 950 6050 50  0001 C CNN
+F 3 "~" H 950 6050 50  0001 C CNN
+	1    950  6050
+	1    0    0    -1
+$EndComp
+$Comp
+L Mechanical:MountingHole H1
+U 1 1 5FEDAB5A
+P 950 5750
+F 0 "H1" H 1050 5795 50  0000 L CNN
+F 1 "MountingHole" H 1050 5706 50  0000 L CNN
+F 2 "MountingHole:MountingHole_2.7mm_M2.5_DIN965" H 950 5750 50  0001 C CNN
+F 3 "~" H 950 5750 50  0001 C CNN
+	1    950  5750
+	1    0    0    -1
+$EndComp
+Wire Wire Line
+	2350 3400 3700 3400
+Wire Wire Line
+	2150 3500 3700 3500
+Wire Wire Line
+	1850 3600 3700 3600
+Wire Wire Line
+	2900 1750 1150 1750
+Wire Wire Line
+	3200 3800 750  3800
+$Comp
+L Connector:Conn_Coaxial J1
+U 1 1 614769F9
+P 2100 5050
+AR Path="/614769F9" Ref="J1"  Part="1"
+AR Path="/61464E7A/614769F9" Ref="J?"  Part="1"
+F 0 "J1" H 2200 5025 50  0000 L CNN
+F 1 "Conn_Coaxial" H 2200 4934 50  0000 L CNN
+F 2 "" H 2100 5050 50  0001 C CNN
+F 3 " ~" H 2100 5050 50  0001 C CNN
+	1    2100 5050
 	-1   0    0    1
 $EndComp
-Wire Wire Line
-	1400 3300 3700 3300
-Wire Wire Line
-	1400 3500 2450 3500
-Wire Wire Line
-	2450 3500 2450 3400
-Wire Wire Line
-	2450 3400 3700 3400
-Wire Wire Line
-	3700 3500 2650 3500
-Wire Wire Line
-	2650 3500 2650 3700
-Wire Wire Line
-	2650 3700 1400 3700
-Wire Wire Line
-	1400 3900 2800 3900
-Wire Wire Line
-	2800 3900 2800 3600
-Wire Wire Line
-	2800 3600 3700 3600
-Wire Wire Line
-	1400 3200 1500 3200
-Wire Wire Line
-	1500 3200 1500 3400
-Wire Wire Line
-	1400 4000 1500 4000
-Connection ~ 1500 4000
-Wire Wire Line
-	1500 4000 1500 4200
-Wire Wire Line
-	1400 3800 1500 3800
-Connection ~ 1500 3800
-Wire Wire Line
-	1500 3800 1500 4000
-Wire Wire Line
-	1400 3600 1500 3600
-Connection ~ 1500 3600
-Wire Wire Line
-	1500 3600 1500 3800
-Wire Wire Line
-	1400 3400 1500 3400
-Connection ~ 1500 3400
-Wire Wire Line
-	1500 3400 1500 3600
+$Comp
+L Logic_LevelTranslator:SN74LV1T34DBV U4
+U 1 1 614769FF
+P 2900 5050
+AR Path="/614769FF" Ref="U4"  Part="1"
+AR Path="/61464E7A/614769FF" Ref="U?"  Part="1"
+F 0 "U4" H 3244 5096 50  0000 L CNN
+F 1 "SN74LV1T34DBV" H 3244 5005 50  0000 L CNN
+F 2 "Package_TO_SOT_SMD:SOT-23-5" H 3550 4800 50  0001 C CNN
+F 3 "https://www.ti.com/lit/ds/symlink/sn74lv1t34.pdf" H 2500 4850 50  0001 C CNN
+	1    2900 5050
+	1    0    0    -1
+$EndComp
+$Comp
+L power:GND #PWR01
+U 1 1 61476A05
+P 2100 4650
+AR Path="/61476A05" Ref="#PWR01"  Part="1"
+AR Path="/61464E7A/61476A05" Ref="#PWR?"  Part="1"
+F 0 "#PWR01" H 2100 4400 50  0001 C CNN
+F 1 "GND" H 2105 4477 50  0000 C CNN
+F 2 "" H 2100 4650 50  0001 C CNN
+F 3 "" H 2100 4650 50  0001 C CNN
+	1    2100 4650
+	-1   0    0    1
+$EndComp
+$Comp
+L power:GND #PWR03
+U 1 1 61476A0B
+P 2900 5550
+AR Path="/61476A0B" Ref="#PWR03"  Part="1"
+AR Path="/61464E7A/61476A0B" Ref="#PWR?"  Part="1"
+F 0 "#PWR03" H 2900 5300 50  0001 C CNN
+F 1 "GND" H 2905 5377 50  0000 C CNN
+F 2 "" H 2900 5550 50  0001 C CNN
+F 3 "" H 2900 5550 50  0001 C CNN
+	1    2900 5550
+	1    0    0    -1
+$EndComp
+Wire Wire Line
+	2100 4850 2100 4650
+Wire Wire Line
+	2900 5350 2900 5550
+Wire Wire Line
+	2300 5050 2600 5050
+Wire Wire Line
+	3200 3800 3200 5050
+NoConn ~ 750  1950
+NoConn ~ 850  1950
+NoConn ~ 950  1950
+NoConn ~ 1050 1950
+NoConn ~ 1250 1950
+NoConn ~ 1350 1950
+NoConn ~ 1450 1950
+NoConn ~ 1550 1950
+NoConn ~ 1650 1950
+NoConn ~ 1750 1950
+NoConn ~ 1850 1950
+NoConn ~ 1950 1950
+NoConn ~ 2050 1950
+NoConn ~ 2150 1950
+NoConn ~ 2250 1950
+NoConn ~ 2350 1950
+NoConn ~ 2450 1950
+NoConn ~ 2550 1950
+NoConn ~ 2650 1950
+NoConn ~ 2550 3300
+NoConn ~ 2450 3300
+NoConn ~ 2250 3300
+NoConn ~ 2050 3300
+NoConn ~ 1950 3300
+NoConn ~ 1750 3300
+NoConn ~ 1650 3300
+NoConn ~ 1550 3300
+NoConn ~ 1350 3300
+NoConn ~ 1250 3300
+NoConn ~ 1150 3300
+NoConn ~ 1050 3300
+NoConn ~ 950  3300
+NoConn ~ 850  3300
+$Comp
+L power:GND #PWR0101
+U 1 1 61497892
+P 1450 3500
+AR Path="/61497892" Ref="#PWR0101"  Part="1"
+AR Path="/61464E7A/61497892" Ref="#PWR?"  Part="1"
+F 0 "#PWR0101" H 1450 3250 50  0001 C CNN
+F 1 "GND" H 1455 3327 50  0000 C CNN
+F 2 "" H 1450 3500 50  0001 C CNN
+F 3 "" H 1450 3500 50  0001 C CNN
+	1    1450 3500
+	1    0    0    -1
+$EndComp
+Wire Wire Line
+	1150 1900 1150 1750
+Wire Wire Line
+	2650 3300 3700 3300
+Wire Wire Line
+	2350 3300 2350 3400
+Wire Wire Line
+	2150 3300 2150 3500
+Wire Wire Line
+	1850 3300 1850 3600
+Wire Wire Line
+	1450 3300 1450 3500
+Wire Wire Line
+	750  3300 750  3800
+Wire Wire Line
+	3100 800  3100 2300
+Wire Wire Line
+	2900 1750 2900 4750
+$Comp
+L MCU_RaspberryPi_and_Boards:Pico U3
+U 1 1 61433A4C
+P 1700 2600
+F 0 "U3" H 1700 3815 50  0000 C CNN
+F 1 "Pico" H 1700 3724 50  0000 C CNN
+F 2 "RPi_Pico:RPi_Pico_SMD_TH" V 1700 2600 50  0001 C CNN
+F 3 "" H 1700 2600 50  0001 C CNN
+	1    1700 2600
+	0    -1   -1   0
+$EndComp
+NoConn ~ 2850 2500
+NoConn ~ 2850 2600
+NoConn ~ 2850 2700
 $EndSCHEMATC
