File: KiCAD/PrawnBlaster.sch (KiCad schematic (older format))
At the start: 16 parts, among them J1 Conn_Coaxial, J11 Flag_12, J5 Flag_14, J8 Flag_13, U3 Pico, U4 SN74LV1T34DBV

Commit message: rearranged input buffer
Parts:
- added H5, H6, H7, H8: MountingHole, MountingHole:MountingHole_2.7mm_M2.5_DIN965, symbol Mechanical:MountingHole
- added J2: Flag_12, Connector_Coaxial:SMA_Amphenol_132134_Vertical, symbol Connector:Conn_Coaxial
- U1: renamed from U3; symbol MCU_RaspberryPi_and_Boards:Pico -> PrawnBlaster-rescue:Pico-MCU_RaspberryPi_and_Boards
- renumbered J5 to J3, J8 to J4, J11 to J5, U4 to U2
Connections:
- wire segments 36 -> 45

Commit message: Add GND connections, update authorship
Connections:
- wire segments 45 -> 54
- no-connect marks 36 -> 29
Changed lines of the file:
@@
 encoding utf-8
 Sheet 1 4
-Title "Prawnblaster Breakout Board, Output Buffers"
+Title "Prawnblaster Breakout Board"
 Date "2020-12-11"
 Rev "v1.0"
 Comp "TU Darmstadt, Institut für Angewandte Physik, AG Birkl"
-Comment1 "Email: patrick.baus@physik.tu-darmstadt.de"
-Comment2 "Design by: Patrick Baus and Lars Pause"
+Comment1 "Email: lars.pause@physik.tu-darmstadt.de"
+Comment2 "Design by: Lars Pause and Eric Bossert"
 Comment3 ""
 Comment4 ""
@@
 NoConn ~ 1850 4500
 NoConn ~ 1850 4400
-NoConn ~ 1850 4300
 NoConn ~ 1850 4200
 NoConn ~ 1850 4000
 NoConn ~ 3250 2700
-NoConn ~ 3250 2800
 NoConn ~ 3250 3000
 NoConn ~ 3250 3200
-NoConn ~ 3250 3300
 NoConn ~ 3250 3500
 NoConn ~ 3250 3600
@@
 NoConn ~ 3250 4100
 NoConn ~ 3250 4200
-NoConn ~ 3250 4300
 NoConn ~ 3250 4400
 $Comp
@@
 	3250 3800 3450 3800
 NoConn ~ 2450 2400
-NoConn ~ 2550 2400
 NoConn ~ 2650 2400
 $Comp
@@
 $EndComp
 NoConn ~ 1850 2700
-NoConn ~ 1850 2800
 NoConn ~ 1850 2900
 NoConn ~ 1850 3000
 NoConn ~ 1850 3100
 NoConn ~ 1850 3200
-NoConn ~ 1850 3300
 NoConn ~ 1850 3400
 NoConn ~ 1850 3500
@@
 NoConn ~ 1850 3900
 Wire Wire Line
-	1700 5500 3200 5500
+	1700 5500 2350 5500
 NoConn ~ 1850 2600
+$Comp
+L power:GND #PWR0101
+U 1 1 614CD6FF
+P 3600 3300
+F 0 "#PWR0101" H 3600 3050 50  0001 C CNN
+F 1 "GND" H 3605 3127 50  0000 C CNN
+F 2 "" H 3600 3300 50  0001 C CNN
+F 3 "" H 3600 3300 50  0001 C CNN
+	1    3600 3300
+	1    0    0    -1
+$EndComp
+$Comp
+L power:GND #PWR0102
+U 1 1 614CE178
+P 3900 2800
+F 0 "#PWR0102" H 3900 2550 50  0001 C CNN
+F 1 "GND" H 3905 2627 50  0000 C CNN
+F 2 "" H 3900 2800 50  0001 C CNN
+F 3 "" H 3900 2800 50  0001 C CNN
+	1    3900 2800
+	1    0    0    -1
+$EndComp
+$Comp
+L power:GND #PWR0103
+U 1 1 614CEAB3
+P 3400 4300
+F 0 "#PWR0103" H 3400 4050 50  0001 C CNN
+F 1 "GND" H 3405 4127 50  0000 C CNN
+F 2 "" H 3400 4300 50  0001 C CNN
+F 3 "" H 3400 4300 50  0001 C CNN
+	1    3400 4300
+	1    0    0    -1
+$EndComp
+$Comp
+L power:GND #PWR0104
+U 1 1 614CED5F
+P 1750 4300
+F 0 "#PWR0104" H 1750 4050 50  0001 C CNN
+F 1 "GND" H 1755 4127 50  0000 C CNN
+F 2 "" H 1750 4300 50  0001 C CNN
+F 3 "" H 1750 4300 50  0001 C CNN
+	1    1750 4300
+	1    0    0    -1
+$EndComp
+$Comp
+L power:GND #PWR0105
+U 1 1 614CF038
+P 1750 3300
+F 0 "#PWR0105" H 1750 3050 50  0001 C CNN
+F 1 "GND" H 1755 3127 50  0000 C CNN
+F 2 "" H 1750 3300 50  0001 C CNN
+F 3 "" H 1750 3300 50  0001 C CNN
+	1    1750 3300
+	1    0    0    -1
+$EndComp
+$Comp
+L power:GND #PWR0106
+U 1 1 614CF31C
+P 1750 2800
+F 0 "#PWR0106" H 1750 2550 50  0001 C CNN
+F 1 "GND" H 1755 2627 50  0000 C CNN
+F 2 "" H 1750 2800 50  0001 C CNN
+F 3 "" H 1750 2800 50  0001 C CNN
+	1    1750 2800
+	1    0    0    -1
+$EndComp
+Wire Wire Line
+	1850 2800 1750 2800
+Wire Wire Line
+	1850 3300 1750 3300
+Wire Wire Line
+	1850 4300 1750 4300
+Wire Wire Line
+	3250 4300 3400 4300
+Wire Wire Line
+	3250 3300 3600 3300
+Wire Wire Line
+	3250 2800 3900 2800
+$Comp
+L power:GND #PWR0107
+U 1 1 614D4FC3
+P 2800 2250
+F 0 "#PWR0107" H 2800 2000 50  0001 C CNN
+F 1 "GND" H 2805 2077 50  0000 C CNN
+F 2 "" H 2800 2250 50  0001 C CNN
+F 3 "" H 2800 2250 50  0001 C CNN
+	1    2800 2250
+	1    0    0    -1
+$EndComp
+Wire Wire Line
+	2550 2400 2550 2250
+Wire Wire Line
+	2550 2250 2800 2250
+$Comp
+L power:PWR_FLAG #FLG0101
+U 1 1 614E9AFB
+P 2350 5500
+F 0 "#FLG0101" H 2350 5575 50  0001 C CNN
+F 1 "PWR_FLAG" H 2350 5673 50  0000 C CNN
+F 2 "" H 2350 5500 50  0001 C CNN
+F 3 "~" H 2350 5500 50  0001 C CNN
+	1    2350 5500
+	1    0    0    -1
+$EndComp
+Connection ~ 2350 5500
+Wire Wire Line
+	2350 5500 3200 5500
 $EndSCHEMATC

Commit message: Add 64Pin Case Power Supply, update PCB dimensions and SMA-Type
Note: Pi Pico footprint is missing!
Parts:
- removed H2, H3, H6, H8: MountingHole, MountingHole:MountingHole_2.7mm_M2.5_DIN965, symbol Mechanical:MountingHole
- J1: footprint (none) -> Connector_Coaxial:SMA_Amphenol_132289_EdgeMount
- J2, J3, J4, J5: footprint Connector_Coaxial:SMA_Amphenol_132134_Vertical -> Connector_Coaxial:SMA_Amphenol_132289_EdgeMount
Changed lines of the file:
@@
 F 0 "J3" H 10310 2970 50  0000 C CNN
 F 1 "Flag_14" V 10410 2790 50  0000 C CNN
-F 2 "Connector_Coaxial:SMA_Amphenol_132134_Vertical" H 10300 2850 50  0001 C CNN
+F 2 "Connector_Coaxial:SMA_Amphenol_132289_EdgeMount" H 10300 2850 50  0001 C CNN
 F 3 "" H 10300 2850 50  0000 C CNN
 F 4 "Molex" H 10300 2850 60  0001 C CNN "MFN"
@@
 F 0 "J4" H 10560 2720 50  0000 C CNN
 F 1 "Flag_13" V 10660 2540 50  0000 C CNN
-F 2 "Connector_Coaxial:SMA_Amphenol_132134_Vertical" H 10550 2600 50  0001 C CNN
+F 2 "Connector_Coaxial:SMA_Amphenol_132289_EdgeMount" H 10550 2600 50  0001 C CNN
 F 3 "" H 10550 2600 50  0000 C CNN
 F 4 "Molex" H 10550 2600 60  0001 C CNN "MFN"
@@
 F 0 "J5" H 10910 2470 50  0000 C CNN
 F 1 "Flag_12" V 11010 2290 50  0000 C CNN
-F 2 "Connector_Coaxial:SMA_Amphenol_132134_Vertical" H 10900 2350 50  0001 C CNN
+F 2 "Connector_Coaxial:SMA_Amphenol_132289_EdgeMount" H 10900 2350 50  0001 C CNN
 F 3 "" H 10900 2350 50  0000 C CNN
 F 4 "Molex" H 10900 2350 60  0001 C CNN "MFN"
@@
 Text Notes 8650 2100 0    60   ~ 0
 Use at least 250 mW resistors!\n(70 mA @ 50 Ω)
-$Comp
-L Mechanical:MountingHole H2
-U 1 1 614A335B
-P 950 5750
-F 0 "H2" H 1050 5795 50  0000 L CNN
-F 1 "MountingHole" H 1050 5706 50  0000 L CNN
-F 2 "MountingHole:MountingHole_2.7mm_M2.5_DIN965" H 950 5750 50  0001 C CNN
-F 3 "~" H 950 5750 50  0001 C CNN
-	1    950  5750
-	1    0    0    -1
-$EndComp
-$Comp
-L Mechanical:MountingHole H3
-U 1 1 5FEDBA18
-P 950 6050
-F 0 "H3" H 1050 6095 50  0000 L CNN
-F 1 "MountingHole" H 1050 6006 50  0000 L CNN
-F 2 "MountingHole:MountingHole_2.7mm_M2.5_DIN965" H 950 6050 50  0001 C CNN
-F 3 "~" H 950 6050 50  0001 C CNN
-	1    950  6050
-	1    0    0    -1
-$EndComp
-$Comp
-L Mechanical:MountingHole H6
-U 1 1 614A335D
-P 950 6350
-F 0 "H6" H 1050 6395 50  0000 L CNN
-F 1 "MountingHole" H 1050 6306 50  0000 L CNN
-F 2 "MountingHole:MountingHole_2.7mm_M2.5_DIN965" H 950 6350 50  0001 C CNN
-F 3 "~" H 950 6350 50  0001 C CNN
-	1    950  6350
-	1    0    0    -1
-$EndComp
-$Comp
-L Mechanical:MountingHole H8
-U 1 1 614A335E
-P 950 6650
-F 0 "H8" H 1050 6695 50  0000 L CNN
-F 1 "MountingHole" H 1050 6606 50  0000 L CNN
-F 2 "MountingHole:MountingHole_2.7mm_M2.5_DIN965" H 950 6650 50  0001 C CNN
-F 3 "~" H 950 6650 50  0001 C CNN
-	1    950  6650
-	1    0    0    -1
-$EndComp
 $Comp
 L Graphic:Logo_Open_Hardware_Small LOGO2
@@
 L Mechanical:MountingHole H7
 U 1 1 5FEDD2EF
-P 950 6650
-F 0 "H7" H 1050 6695 50  0000 L CNN
-F 1 "MountingHole" H 1050 6606 50  0000 L CNN
-F 2 "MountingHole:MountingHole_2.7mm_M2.5_DIN965" H 950 6650 50  0001 C CNN
-F 3 "~" H 950 6650 50  0001 C CNN
-	1    950  6650
+P 850 6700
+F 0 "H7" H 950 6745 50  0000 L CNN
+F 1 "MountingHole" H 950 6656 50  0000 L CNN
+F 2 "MountingHole:MountingHole_2.7mm_M2.5_DIN965" H 850 6700 50  0001 C CNN
+F 3 "~" H 850 6700 50  0001 C CNN
+	1    850  6700
 	1    0    0    -1
 $EndComp
@@
 L Mechanical:MountingHole H5
 U 1 1 5FEDC6AA
-P 950 6350
-F 0 "H5" H 1050 6395 50  0000 L CNN
-F 1 "MountingHole" H 1050 6306 50  0000 L CNN
-F 2 "MountingHole:MountingHole_2.7mm_M2.5_DIN965" H 950 6350 50  0001 C CNN
-F 3 "~" H 950 6350 50  0001 C CNN
-	1    950  6350
+P 850 6400
+F 0 "H5" H 950 6445 50  0000 L CNN
+F 1 "MountingHole" H 950 6356 50  0000 L CNN
+F 2 "MountingHole:MountingHole_2.7mm_M2.5_DIN965" H 850 6400 50  0001 C CNN
+F 3 "~" H 850 6400 50  0001 C CNN
+	1    850  6400
 	1    0    0    -1
 $EndComp
@@
 L Mechanical:MountingHole H4
 U 1 1 614A335C
-P 950 6050
-F 0 "H4" H 1050 6095 50  0000 L CNN
-F 1 "MountingHole" H 1050 6006 50  0000 L CNN
-F 2 "MountingHole:MountingHole_2.7mm_M2.5_DIN965" H 950 6050 50  0001 C CNN
-F 3 "~" H 950 6050 50  0001 C CNN
-	1    950  6050
+P 850 6100
+F 0 "H4" H 950 6145 50  0000 L CNN
+F 1 "MountingHole" H 950 6056 50  0000 L CNN
+F 2 "MountingHole:MountingHole_2.7mm_M2.5_DIN965" H 850 6100 50  0001 C CNN
+F 3 "~" H 850 6100 50  0001 C CNN
+	1    850  6100
 	1    0    0    -1
 $EndComp
@@
 L Mechanical:MountingHole H1
 U 1 1 5FEDAB5A
-P 950 5750
-F 0 "H1" H 1050 5795 50  0000 L CNN
-F 1 "MountingHole" H 1050 5706 50  0000 L CNN
-F 2 "MountingHole:MountingHole_2.7mm_M2.5_DIN965" H 950 5750 50  0001 C CNN
-F 3 "~" H 950 5750 50  0001 C CNN
-	1    950  5750
+P 850 5800
+F 0 "H1" H 950 5845 50  0000 L CNN
+F 1 "MountingHole" H 950 5756 50  0000 L CNN
+F 2 "MountingHole:MountingHole_2.7mm_M2.5_DIN965" H 850 5800 50  0001 C CNN
+F 3 "~" H 850 5800 50  0001 C CNN
+	1    850  5800
 	1    0    0    -1
 $EndComp
@@
 F 0 "J2" H 10060 3220 50  0000 C CNN
 F 1 "Flag_12" V 10160 3040 50  0000 C CNN
-F 2 "Connector_Coaxial:SMA_Amphenol_132134_Vertical" H 10050 3100 50  0001 C CNN
+F 2 "Connector_Coaxial:SMA_Amphenol_132289_EdgeMount" H 10050 3100 50  0001 C CNN
 F 3 "" H 10050 3100 50  0000 C CNN
 F 4 "Molex" H 10050 3100 60  0001 C CNN "MFN"
@@
 F 0 "J1" H 2500 6475 50  0000 L CNN
 F 1 "Conn_Coaxial" H 2500 6384 50  0000 L CNN
-F 2 "" H 2400 6500 50  0001 C CNN
+F 2 "Connector_Coaxial:SMA_Amphenol_132289_EdgeMount" H 2400 6500 50  0001 C CNN
 F 3 " ~" H 2400 6500 50  0001 C CNN
 	1    2400 6500

Commit message: added clock input
Parts:
- added J7: Conn_Coaxial, Connector_Coaxial:SMA_Amphenol_132289_EdgeMount, symbol Connector:Conn_Coaxial
- added U5: SN74LV1T34DBV, Package_TO_SOT_SMD:SOT-23-5, symbol Logic_LevelTranslator:SN74LV1T34DBV
Connections:
- wire segments 54 -> 63
- no-connect marks 29 -> 28
Other:
- note added: "Clock input"
- note added: "External trigger input"
Changed lines of the file:
@@
 NoConn ~ 1850 2900
 NoConn ~ 1850 3000
-NoConn ~ 1850 3100
 NoConn ~ 1850 3200
 NoConn ~ 1850 3400
@@
 Wire Wire Line
 	2350 5500 3200 5500
+$Comp
+L Connector:Conn_Coaxial J7
+U 1 1 6158A65F
+P 4800 6500
+AR Path="/6158A65F" Ref="J7"  Part="1"
+AR Path="/61464E7A/6158A65F" Ref="J?"  Part="1"
+F 0 "J7" H 4900 6475 50  0000 L CNN
+F 1 "Conn_Coaxial" H 4900 6384 50  0000 L CNN
+F 2 "Connector_Coaxial:SMA_Amphenol_132289_EdgeMount" H 4800 6500 50  0001 C CNN
+F 3 " ~" H 4800 6500 50  0001 C CNN
+	1    4800 6500
+	-1   0    0    1
+$EndComp
+$Comp
+L Logic_LevelTranslator:SN74LV1T34DBV U5
+U 1 1 6158A665
+P 5600 6500
+AR Path="/6158A665" Ref="U5"  Part="1"
+AR Path="/61464E7A/6158A665" Ref="U?"  Part="1"
+F 0 "U5" H 5944 6546 50  0000 L CNN
+F 1 "SN74LV1T34DBV" H 5944 6455 50  0000 L CNN
+F 2 "Package_TO_SOT_SMD:SOT-23-5" H 6250 6250 50  0001 C CNN
+F 3 "https://www.ti.com/lit/ds/symlink/sn74lv1t34.pdf" H 5200 6300 50  0001 C CNN
+	1    5600 6500
+	1    0    0    -1
+$EndComp
+$Comp
+L power:GND #PWR022
+U 1 1 6158A66B
+P 4800 6100
+AR Path="/6158A66B" Ref="#PWR022"  Part="1"
+AR Path="/61464E7A/6158A66B" Ref="#PWR?"  Part="1"
+F 0 "#PWR022" H 4800 5850 50  0001 C CNN
+F 1 "GND" H 4805 5927 50  0000 C CNN
+F 2 "" H 4800 6100 50  0001 C CNN
+F 3 "" H 4800 6100 50  0001 C CNN
+	1    4800 6100
+	-1   0    0    1
+$EndComp
+$Comp
+L power:GND #PWR023
+U 1 1 6158A671
+P 5600 7000
+AR Path="/6158A671" Ref="#PWR023"  Part="1"
+AR Path="/61464E7A/6158A671" Ref="#PWR?"  Part="1"
+F 0 "#PWR023" H 5600 6750 50  0001 C CNN
+F 1 "GND" H 5605 6827 50  0000 C CNN
+F 2 "" H 5600 7000 50  0001 C CNN
+F 3 "" H 5600 7000 50  0001 C CNN
+	1    5600 7000
+	1    0    0    -1
+$EndComp
+Wire Wire Line
+	4800 6300 4800 6100
+Wire Wire Line
+	5600 6800 5600 7000
+Wire Wire Line
+	5000 6500 5300 6500
+Wire Wire Line
+	5600 5500 5600 6200
+Connection ~ 3200 5500
+Wire Wire Line
+	1850 3100 1400 3100
+Wire Wire Line
+	1400 3100 1400 4950
+Wire Wire Line
+	1400 4950 5900 4950
+Wire Wire Line
+	5900 4950 5900 6500
+Wire Wire Line
+	3200 5500 5600 5500
+Text Notes 4600 6700 0    50   ~ 0
+Clock input
+Text Notes 2100 6750 0    50   ~ 0
+External trigger input
 $EndSCHEMATC

Commit message: Add PiPico Footprint and route PCB without SMA connectors
Schematic was updated and routing on PCB was done except for input/output connectors.
Parts:
- added J10, J8: Conn_01x20_Male, Connector_PinHeader_2.54mm:PinHeader_1x20_P2.54mm_Vertical, symbol Connector:Conn_01x20_Male
- added J9: Conn_01x03_Male, Connector_PinHeader_2.54mm:PinHeader_1x03_P2.54mm_Vertical, symbol Connector:Conn_01x03_Male
- U1: footprint RPi_Pico:RPi_Pico_SMD_TH -> Custom_footprints_project:RPi_Pico_SMD_TH
Connections:
- wire segments 63 -> 102
- no-connect marks 28 -> 0

Commit message: Exchange SMA-connectors with pin-header
Add pin Header to connect PCB with new Frontpanel PCB. Necessary distances marked. Routing finished.
Parts:
- removed J1, J7: Conn_Coaxial, Connector_Coaxial:SMA_Amphenol_132289_EdgeMount, symbol Connector:Conn_Coaxial
- removed J2, J5: Flag_12, Connector_Coaxial:SMA_Amphenol_132289_EdgeMount, symbol Connector:Conn_Coaxial
- removed J3: Flag_14, Connector_Coaxial:SMA_Amphenol_132289_EdgeMount, symbol Connector:Conn_Coaxial
- removed J4: Flag_13, Connector_Coaxial:SMA_Amphenol_132289_EdgeMount, symbol Connector:Conn_Coaxial
- added J1: Conn_02x06_Odd_Even, Connector_PinSocket_2.54mm:PinSocket_2x06_P2.54mm_Horizontal, symbol Connector_Generic:Conn_02x06_Odd_Even
Connections:
- wire segments 102 -> 113
Other:
- note removed: "Clock input"
- note removed: "External trigger input"
