File: KiCAD/PrawnBlaster.sch (KiCad schematic (older format))
At the start: 17 parts, among them J1 Conn_02x06_Odd_Even, J10 Conn_01x20_Male, J8 Conn_01x20_Male, J9 Conn_01x03_Male, U1 Pico, U2 SN74LV1T34DBV, U5 SN74LV1T34DBV

Commit message: Finish routing PCB
Parts:
- removed H1, H4, H5, H7: MountingHole, MountingHole:MountingHole_2.7mm_M2.5_DIN965, symbol Mechanical:MountingHole
- added C5: 100n, Capacitor_SMD:C_0603_1608Metric, symbol Device:C
- added C6: 10u, Capacitor_SMD:C_1210_3225Metric, symbol Device:C
Connections:
- wire segments 113 -> 120
Changed lines of the file:
@@
-$EndComp
-$Comp
-L Mechanical:MountingHole H7
-U 1 1 5FEDD2EF
-P 850 6700
-F 0 "H7" H 950 6745 50  0000 L CNN
-F 1 "MountingHole" H 950 6656 50  0000 L CNN
-F 2 "MountingHole:MountingHole_2.7mm_M2.5_DIN965" H 850 6700 50  0001 C CNN
-F 3 "~" H 850 6700 50  0001 C CNN
-	1    850  6700
-	1    0    0    -1
-$EndComp
-$Comp
-L Mechanical:MountingHole H5
-U 1 1 5FEDC6AA
-P 850 6400
-F 0 "H5" H 950 6445 50  0000 L CNN
-F 1 "MountingHole" H 950 6356 50  0000 L CNN
-F 2 "MountingHole:MountingHole_2.7mm_M2.5_DIN965" H 850 6400 50  0001 C CNN
-F 3 "~" H 850 6400 50  0001 C CNN
-	1    850  6400
-	1    0    0    -1
-$EndComp
-$Comp
-L Mechanical:MountingHole H4
-U 1 1 614A335C
-P 850 6100
-F 0 "H4" H 950 6145 50  0000 L CNN
-F 1 "MountingHole" H 950 6056 50  0000 L CNN
-F 2 "MountingHole:MountingHole_2.7mm_M2.5_DIN965" H 850 6100 50  0001 C CNN
-F 3 "~" H 850 6100 50  0001 C CNN
-	1    850  6100
-	1    0    0    -1
-$EndComp
-$Comp
-L Mechanical:MountingHole H1
-U 1 1 5FEDAB5A
-P 850 5800
-F 0 "H1" H 950 5845 50  0000 L CNN
-F 1 "MountingHole" H 950 5756 50  0000 L CNN
-F 2 "MountingHole:MountingHole_2.7mm_M2.5_DIN965" H 850 5800 50  0001 C CNN
-F 3 "~" H 850 5800 50  0001 C CNN
-	1    850  5800
-	1    0    0    -1
 $EndComp
 $Comp
@@
 	1550 4950 7100 4950
 Wire Wire Line
-	6600 5300 6600 4000
-Wire Wire Line
-	6600 4000 6800 4000
-Connection ~ 6600 5300
-Wire Wire Line
-	6600 5300 6800 5300
+	6200 5300 6200 4350
+Wire Wire Line
+	6200 4000 6800 4000
+Connection ~ 6200 5300
+Wire Wire Line
+	6200 5300 6800 5300
 Wire Wire Line
 	7400 5300 7500 5300
@@
 	7050 1800 7900 1800
 Wire Wire Line
-	8200 1800 8950 1800
-Wire Wire Line
 	7050 1900 8100 1900
 Wire Wire Line
-	8400 1900 8950 1900
-Wire Wire Line
 	7050 2000 7850 2000
 Wire Wire Line
-	8150 2000 8950 2000
-Wire Wire Line
 	7050 2100 8100 2100
 Wire Wire Line
-	8400 2100 8950 2100
-Wire Wire Line
 	7100 4300 7100 4350
 Wire Wire Line
@@
 	7100 5700 8600 5700
 Wire Wire Line
-	2350 5300 6600 5300
+	2350 5300 6200 5300
 $Sheet
 S 5650 700  1400 1950
@@
 F1 "output_buffer.sch" 60
 F2 "Vcc" U L 5650 800 60
-F3 "A0" I L 5650 1800 50
-F4 "A1" I L 5650 1900 50
-F5 "A2" I L 5650 2000 50
-F6 "A3" I L 5650 2100 50
-F7 "B0" O R 7050 1800 50
-F8 "B1" O R 7050 1900 50
-F9 "B2" O R 7050 2000 50
-F10 "B3" O R 7050 2100 50
+F3 "A0" I L 5650 2100 50
+F4 "A1" I L 5650 2000 50
+F5 "A2" I L 5650 1900 50
+F6 "A3" I L 5650 1800 50
+F7 "B0" O R 7050 2100 50
+F8 "B1" O R 7050 2000 50
+F9 "B2" O R 7050 1900 50
+F10 "B3" O R 7050 1800 50
 $EndSheet
-Wire Wire Line
-	8600 5700 8600 1600
-Wire Wire Line
-	8600 1600 8950 1600
-Wire Wire Line
-	8450 4350 8450 1700
-Wire Wire Line
-	8450 1700 8950 1700
+Wire Notes Line
+	9150 1400 9550 1400
+Text Notes 7150 1450 0    60   ~ 0
+Use at least 250 mW resistors!\n(70 mA @ 50 Ω)
+Wire Wire Line
+	3250 3100 3550 3100
+Wire Wire Line
+	3250 3400 3450 3400
+Wire Wire Line
+	3650 2000 3650 2900
+Wire Wire Line
+	3750 2100 3750 2600
+Wire Wire Line
+	8400 1900 8950 1900
+Wire Wire Line
+	8200 1800 8950 1800
+Wire Wire Line
+	8400 2100 8950 2100
+Wire Wire Line
+	8150 2000 8950 2000
+Wire Wire Line
+	9450 2100 9500 2100
+Wire Wire Line
+	9500 2100 9500 2150
+Wire Wire Line
+	9450 2000 9600 2000
+Wire Wire Line
+	9600 2000 9600 2050
+Wire Wire Line
+	9450 1900 9700 1900
+Wire Wire Line
+	9700 1900 9700 1950
+Wire Wire Line
+	9450 1800 9800 1800
+Wire Wire Line
+	9800 1800 9800 1850
+Wire Wire Line
+	9450 1700 9900 1700
+Wire Wire Line
+	9900 1700 9900 1750
+Wire Wire Line
+	9450 1600 10000 1600
+Wire Wire Line
+	10000 1600 10000 1650
+$Comp
+L power:GND #PWR0110
+U 1 1 616E7065
+P 10000 1650
+F 0 "#PWR0110" H 10000 1400 50  0001 C CNN
+F 1 "GND" H 10005 1477 50  0000 C CNN
+F 2 "" H 10000 1650 50  0001 C CNN
+F 3 "" H 10000 1650 50  0001 C CNN
+	1    10000 1650
+	1    0    0    -1
+$EndComp
+$Comp
+L power:GND #PWR0111
+U 1 1 616E75A8
+P 9900 1750
+F 0 "#PWR0111" H 9900 1500 50  0001 C CNN
+F 1 "GND" H 9905 1577 50  0000 C CNN
+F 2 "" H 9900 1750 50  0001 C CNN
+F 3 "" H 9900 1750 50  0001 C CNN
+	1    9900 1750
+	1    0    0    -1
+$EndComp
+$Comp
+L power:GND #PWR0112
+U 1 1 616E795B
+P 9800 1850
+F 0 "#PWR0112" H 9800 1600 50  0001 C CNN
+F 1 "GND" H 9805 1677 50  0000 C CNN
+F 2 "" H 9800 1850 50  0001 C CNN
+F 3 "" H 9800 1850 50  0001 C CNN
+	1    9800 1850
+	1    0    0    -1
+$EndComp
+$Comp
+L power:GND #PWR0113
+U 1 1 616E7D61
+P 9700 1950
+F 0 "#PWR0113" H 9700 1700 50  0001 C CNN
+F 1 "GND" H 9705 1777 50  0000 C CNN
+F 2 "" H 9700 1950 50  0001 C CNN
+F 3 "" H 9700 1950 50  0001 C CNN
+	1    9700 1950
+	1    0    0    -1
+$EndComp
+$Comp
+L power:GND #PWR0114
+U 1 1 616E8122
+P 9600 2050
+F 0 "#PWR0114" H 9600 1800 50  0001 C CNN
+F 1 "GND" H 9605 1877 50  0000 C CNN
+F 2 "" H 9600 2050 50  0001 C CNN
+F 3 "" H 9600 2050 50  0001 C CNN
+	1    9600 2050
+	1    0    0    -1
+$EndComp
 $Comp
 L power:GND #PWR0115
@@
 	1    0    0    -1
 $EndComp
-$Comp
-L power:GND #PWR0114
-U 1 1 616E8122
-P 9600 2050
-F 0 "#PWR0114" H 9600 1800 50  0001 C CNN
-F 1 "GND" H 9605 1877 50  0000 C CNN
-F 2 "" H 9600 2050 50  0001 C CNN
-F 3 "" H 9600 2050 50  0001 C CNN
-	1    9600 2050
-	1    0    0    -1
-$EndComp
-$Comp
-L power:GND #PWR0113
-U 1 1 616E7D61
-P 9700 1950
-F 0 "#PWR0113" H 9700 1700 50  0001 C CNN
-F 1 "GND" H 9705 1777 50  0000 C CNN
-F 2 "" H 9700 1950 50  0001 C CNN
-F 3 "" H 9700 1950 50  0001 C CNN
-	1    9700 1950
-	1    0    0    -1
-$EndComp
-$Comp
-L power:GND #PWR0112
-U 1 1 616E795B
-P 9800 1850
-F 0 "#PWR0112" H 9800 1600 50  0001 C CNN
-F 1 "GND" H 9805 1677 50  0000 C CNN
-F 2 "" H 9800 1850 50  0001 C CNN
-F 3 "" H 9800 1850 50  0001 C CNN
-	1    9800 1850
-	1    0    0    -1
-$EndComp
-$Comp
-L power:GND #PWR0111
-U 1 1 616E75A8
-P 9900 1750
-F 0 "#PWR0111" H 9900 1500 50  0001 C CNN
-F 1 "GND" H 9905 1577 50  0000 C CNN
-F 2 "" H 9900 1750 50  0001 C CNN
-F 3 "" H 9900 1750 50  0001 C CNN
-	1    9900 1750
-	1    0    0    -1
-$EndComp
-$Comp
-L power:GND #PWR0110
-U 1 1 616E7065
-P 10000 1650
-F 0 "#PWR0110" H 10000 1400 50  0001 C CNN
-F 1 "GND" H 10005 1477 50  0000 C CNN
-F 2 "" H 10000 1650 50  0001 C CNN
-F 3 "" H 10000 1650 50  0001 C CNN
-	1    10000 1650
-	1    0    0    -1
-$EndComp
-Wire Wire Line
-	10000 1600 10000 1650
-Wire Wire Line
-	9450 1600 10000 1600
-Wire Wire Line
-	9900 1700 9900 1750
-Wire Wire Line
-	9450 1700 9900 1700
-Wire Wire Line
-	9800 1800 9800 1850
-Wire Wire Line
-	9450 1800 9800 1800
-Wire Wire Line
-	9700 1900 9700 1950
-Wire Wire Line
-	9450 1900 9700 1900
-Wire Wire Line
-	9600 2000 9600 2050
-Wire Wire Line
-	9450 2000 9600 2000
-Wire Wire Line
-	9500 2100 9500 2150
-Wire Wire Line
-	9450 2100 9500 2100
-Wire Notes Line
-	9150 1400 9550 1400
-Text Notes 7150 1450 0    60   ~ 0
-Use at least 250 mW resistors!\n(70 mA @ 50 Ω)
+Wire Wire Line
+	8600 1600 8950 1600
+Wire Wire Line
+	8600 5700 8600 1600
+Wire Wire Line
+	8450 4350 8450 1700
+Wire Wire Line
+	8450 1700 8950 1700
 $Comp
 L Connector_Generic:Conn_02x06_Odd_Even J1
@@
 	1    0    0    -1
 $EndComp
-Wire Wire Line
-	3250 2600 3450 2600
-Wire Wire Line
-	3250 3100 3650 3100
-Wire Wire Line
-	3250 3400 3750 3400
-Wire Wire Line
-	3450 1800 3450 2600
-Connection ~ 3450 2600
-Wire Wire Line
-	3450 2600 4100 2600
-Wire Wire Line
-	3550 1900 3550 2900
-Wire Wire Line
-	3250 2900 3550 2900
-Connection ~ 3550 2900
-Wire Wire Line
-	3550 2900 4100 2900
-Wire Wire Line
-	3650 2000 3650 3100
-Connection ~ 3650 3100
-Wire Wire Line
-	3650 3100 4100 3100
-Wire Wire Line
-	3750 2100 3750 3400
-Connection ~ 3750 3400
-Wire Wire Line
-	3750 3400 4100 3400
+Connection ~ 3450 3400
+Connection ~ 3550 3100
+Connection ~ 3650 2900
+Wire Wire Line
+	3650 2900 4100 2900
+Connection ~ 3750 2600
+Wire Wire Line
+	3750 2600 4100 2600
+Wire Wire Line
+	3450 3400 4100 3400
+Wire Wire Line
+	3550 3100 4100 3100
+Wire Wire Line
+	3550 1900 3550 3100
+Wire Wire Line
+	3250 2900 3650 2900
+Wire Wire Line
+	3250 2600 3750 2600
+Wire Wire Line
+	3450 1800 3450 3400
+$Comp
+L Device:C C?
+U 1 1 616226E5
+P 6500 4550
+AR Path="/5859B68B/616226E5" Ref="C?"  Part="1"
+AR Path="/616226E5" Ref="C5"  Part="1"
+F 0 "C5" H 6525 4650 50  0000 L CNN
+F 1 "100n" H 6525 4450 50  0000 L CNN
+F 2 "Capacitor_SMD:C_0603_1608Metric" H 6538 4400 50  0001 C CNN
+F 3 "" H 6500 4550 50  0000 C CNN
+F 4 "Kemet" H 6500 4550 60  0001 C CNN "MFN"
+F 5 "C0603C104K3RACTU" H 6500 4550 50  0001 C CNN "PN"
+	1    6500 4550
+	1    0    0    -1
+$EndComp
+$Comp
+L Device:C C?
+U 1 1 616226ED
+P 6800 4550
+AR Path="/5859B68B/616226ED" Ref="C?"  Part="1"
+AR Path="/616226ED" Ref="C6"  Part="1"
+F 0 "C6" H 6825 4650 50  0000 L CNN
+F 1 "10u" H 6825 4450 50  0000 L CNN
+F 2 "Capacitor_SMD:C_1210_3225Metric" H 6838 4400 50  0001 C CNN
+F 3 "" H 6800 4550 50  0000 C CNN
+F 4 "Murata" H 6800 4550 60  0001 C CNN "MFN"
+F 5 "GRM32ER71H106KA12L" H 6800 4550 50  0001 C CNN "PN"
+	1    6800 4550
+	1    0    0    -1
+$EndComp
+Wire Wire Line
+	6500 4750 6500 4700
+Wire Wire Line
+	6200 4350 6500 4350
+Wire Wire Line
+	6500 4350 6500 4400
+Wire Wire Line
+	6800 4350 6800 4400
+Connection ~ 6500 4350
+Wire Wire Line
+	6800 4700 6800 4750
+Wire Wire Line
+	6500 4350 6800 4350
+Connection ~ 6200 4350
+Wire Wire Line
+	6200 4350 6200 4000
+$Comp
+L power:GND #PWR02
+U 1 1 6163D5A5
+P 6500 4750
+F 0 "#PWR02" H 6500 4500 50  0001 C CNN
+F 1 "GND" H 6505 4577 50  0000 C CNN
+F 2 "" H 6500 4750 50  0001 C CNN
+F 3 "" H 6500 4750 50  0001 C CNN
+	1    6500 4750
+	1    0    0    -1
+$EndComp
+$Comp
+L power:GND #PWR03
+U 1 1 6163DB03
+P 6800 4750
+F 0 "#PWR03" H 6800 4500 50  0001 C CNN
+F 1 "GND" H 6805 4577 50  0000 C CNN
+F 2 "" H 6800 4750 50  0001 C CNN
+F 3 "" H 6800 4750 50  0001 C CNN
+	1    6800 4750
+	1    0    0    -1
+$EndComp
 $EndSCHEMATC

Commit message: Update MFN, PN and BOM
Parts:
- J1: MFN (none) -> Samtec; PN (none) -> SSW-106-02-G-D-RA
- J10, J8: MFN (none) -> Samtec; PN (none) -> TSW-120-07-G-S
- J9: MFN (none) -> Samtec; PN (none) -> TSW-103-07-G-S
- R4: MFN (none) -> Panasonic; PN (none) -> ERJ8ENF49R9V
- U1: MFN (none) -> Seeed Studio; PN (none) -> 102110537
- U2, U5: MFN (none) -> Texas Instruments; PN (none) -> SN74LV1T34DBVR
Changed lines of the file:
@@
 F 2 "Package_TO_SOT_SMD:SOT-23-5" H 7750 3750 50  0001 C CNN
 F 3 "https://www.ti.com/lit/ds/symlink/sn74lv1t34.pdf" H 6700 3800 50  0001 C CNN
+F 4 "Texas Instruments" H 7100 4000 50  0001 C CNN "MFN"
+F 5 "SN74LV1T34DBVR" H 7100 4000 50  0001 C CNN "PN"
 	1    7100 4000
 	0    -1   -1   0
@@
 F 2 "Custom_footprints_project:RPi_Pico_SMD_TH" V 2550 3550 50  0001 C CNN
 F 3 "" H 2550 3550 50  0001 C CNN
+F 4 "Seeed Studio" H 2550 3550 50  0001 C CNN "MFN"
+F 5 "102110537" H 2550 3550 50  0001 C CNN "PN"
 	1    2550 3550
 	-1   0    0    1
@@
 F 2 "Package_TO_SOT_SMD:SOT-23-5" H 7750 5050 50  0001 C CNN
 F 3 "https://www.ti.com/lit/ds/symlink/sn74lv1t34.pdf" H 6700 5100 50  0001 C CNN
+F 4 "Texas Instruments" H 7100 5300 50  0001 C CNN "MFN"
+F 5 "SN74LV1T34DBVR" H 7100 5300 50  0001 C CNN "PN"
 	1    7100 5300
 	0    -1   -1   0
@@
 F 2 "Connector_PinHeader_2.54mm:PinHeader_1x20_P2.54mm_Vertical" H 1000 3500 50  0001 C CNN
 F 3 "~" H 1000 3500 50  0001 C CNN
+F 4 "Samtec" H 1000 3500 50  0001 C CNN "MFN"
+F 5 "TSW-120-07-G-S" H 1000 3500 50  0001 C CNN "PN"
 	1    1000 3500
 	1    0    0    -1
@@
 F 2 "Connector_PinHeader_2.54mm:PinHeader_1x20_P2.54mm_Vertical" H 4300 3600 50  0001 C CNN
 F 3 "~" H 4300 3600 50  0001 C CNN
+F 4 "Samtec" H 4300 3600 50  0001 C CNN "MFN"
+F 5 "TSW-120-07-G-S" H 4300 3600 50  0001 C CNN "PN"
 	1    4300 3600
 	-1   0    0    1
@@
 F 2 "Connector_PinHeader_2.54mm:PinHeader_1x03_P2.54mm_Vertical" H 2550 1800 50  0001 C CNN
 F 3 "~" H 2550 1800 50  0001 C CNN
+F 4 "Samtec" H 2550 1800 50  0001 C CNN "MFN"
+F 5 "TSW-103-07-G-S" H 2550 1800 50  0001 C CNN "PN"
 	1    2550 1800
 	0    1    1    0
@@
 F 2 "Resistor_SMD:R_1206_3216Metric" V 8180 2100 50  0001 C CNN
 F 3 "" H 8250 2100 50  0000 C CNN
+F 4 "Panasonic" H 8250 2100 50  0001 C CNN "MFN"
+F 5 "ERJ8ENF49R9V" H 8250 2100 50  0001 C CNN "PN"
 	1    8250 2100
 	0    -1   -1   0
@@
 F 2 "Connector_PinSocket_2.54mm:PinSocket_2x06_P2.54mm_Horizontal" H 9150 1800 50  0001 C CNN
 F 3 "~" H 9150 1800 50  0001 C CNN
+F 4 "Samtec" H 9150 1800 50  0001 C CNN "MFN"
+F 5 "SSW-106-02-G-D-RA" H 9150 1800 50  0001 C CNN "PN"
 	1    9150 1800
 	1    0    0    -1
