File: KiCAD/PrawnBlaster.sch (KiCad schematic (older format))
At the start: 15 parts, among them J1 Conn_02x06_Odd_Even, J10 Conn_01x20_Male, J8 Conn_01x20_Male, J9 Conn_01x03_Male, U1 Pico, U2 SN74LV1T34DBV, U5 SN74LV1T34DBV

Commit message: Add USB-isolator plus extra power supply; move parts
Parts:
- added D3: D_Schottky, Diode_SMD:D_SMA, symbol Device:D_Schottky
- added JP1: Jumper_NO_Small, Jumper:SolderJumper-2_P1.3mm_Open_Pad1.0x1.5mm, symbol Device:Jumper_NO_Small
- added R10, R11: 500, Resistor_SMD:R_0603_1608Metric, symbol Device:R
- added R16, R17: 47k, Resistor_SMD:R_0805_2012Metric, symbol Device:R
- C6: value 10u -> 100n; footprint Capacitor_SMD:C_1210_3225Metric -> Capacitor_SMD:C_0603_1608Metric; MFN Murata -> Kemet; PN GRM32ER71H106KA12L -> C0603C104K3RACTU
- U2, U5: value SN74LV1T34DBV -> 74LVC1G07; MFN Texas Instruments -> Nexperia; PN SN74LV1T34DBVR -> 74LVC1G07GV
Connections:
- net labels added: 3_3V_Pico, adafruit_usb_isolator
- wire segments 120 -> 130

Commit message: Reduce GND-connections to pico to 1
Connections:
- wire segments 130 -> 122
Changed lines of the file:
@@
-	1    0    0    -1
-$EndComp
-$Comp
-L power:GND #PWR01
-U 1 1 61497892
-P 3950 3800
-AR Path="/61497892" Ref="#PWR01"  Part="1"
-AR Path="/61464E7A/61497892" Ref="#PWR?"  Part="1"
-F 0 "#PWR01" H 3950 3550 50  0001 C CNN
-F 1 "GND" H 3955 3627 50  0000 C CNN
-F 2 "" H 3950 3800 50  0001 C CNN
-F 3 "" H 3950 3800 50  0001 C CNN
-	1    3950 3800
 	1    0    0    -1
 $EndComp
 Wire Wire Line
 	1850 4100 1700 4100
-Wire Wire Line
-	3250 3800 3950 3800
 $Comp
 L Logic_LevelTranslator:SN74LV1T34DBV U2
@@
 	1700 5300 1900 5300
 $Comp
-L power:GND #PWR0101
-U 1 1 614CD6FF
-P 3950 3300
-F 0 "#PWR0101" H 3950 3050 50  0001 C CNN
-F 1 "GND" H 3955 3127 50  0000 C CNN
-F 2 "" H 3950 3300 50  0001 C CNN
-F 3 "" H 3950 3300 50  0001 C CNN
-	1    3950 3300
-	1    0    0    -1
-$EndComp
-$Comp
-L power:GND #PWR0102
-U 1 1 614CE178
-P 3950 2800
-F 0 "#PWR0102" H 3950 2550 50  0001 C CNN
-F 1 "GND" H 3955 2627 50  0000 C CNN
-F 2 "" H 3950 2800 50  0001 C CNN
-F 3 "" H 3950 2800 50  0001 C CNN
-	1    3950 2800
-	1    0    0    -1
-$EndComp
-$Comp
-L power:GND #PWR0103
-U 1 1 614CEAB3
-P 3400 4300
-F 0 "#PWR0103" H 3400 4050 50  0001 C CNN
-F 1 "GND" H 3405 4127 50  0000 C CNN
-F 2 "" H 3400 4300 50  0001 C CNN
-F 3 "" H 3400 4300 50  0001 C CNN
-	1    3400 4300
-	1    0    0    -1
-$EndComp
-$Comp
 L power:GND #PWR0104
 U 1 1 614CED5F
@@
 	1    0    0    -1
 $EndComp
-$Comp
-L power:GND #PWR0105
-U 1 1 614CF038
-P 1750 3300
-F 0 "#PWR0105" H 1750 3050 50  0001 C CNN
-F 1 "GND" H 1755 3127 50  0000 C CNN
-F 2 "" H 1750 3300 50  0001 C CNN
-F 3 "" H 1750 3300 50  0001 C CNN
-	1    1750 3300
-	1    0    0    -1
-$EndComp
-$Comp
-L power:GND #PWR0106
-U 1 1 614CF31C
-P 1750 2800
-F 0 "#PWR0106" H 1750 2550 50  0001 C CNN
-F 1 "GND" H 1755 2627 50  0000 C CNN
-F 2 "" H 1750 2800 50  0001 C CNN
-F 3 "" H 1750 2800 50  0001 C CNN
-	1    1750 2800
-	1    0    0    -1
-$EndComp
-Wire Wire Line
-	1850 2800 1750 2800
-Wire Wire Line
-	1850 3300 1750 3300
 Wire Wire Line
 	1850 4300 1750 4300
-Wire Wire Line
-	3250 4300 3400 4300
-Wire Wire Line
-	3250 3300 3950 3300
-Wire Wire Line
-	3250 2800 3950 2800
-$Comp
-L power:GND #PWR0107
-U 1 1 614D4FC3
-P 2800 2250
-F 0 "#PWR0107" H 2800 2000 50  0001 C CNN
-F 1 "GND" H 2805 2077 50  0000 C CNN
-F 2 "" H 2800 2250 50  0001 C CNN
-F 3 "" H 2800 2250 50  0001 C CNN
-	1    2800 2250
-	1    0    0    -1
-$EndComp
-Wire Wire Line
-	2550 2400 2550 2250
-Wire Wire Line
-	2550 2250 2800 2250
 $Comp
 L power:PWR_FLAG #FLG0101
@@
 $EndComp
 Wire Wire Line
-	4100 2800 3950 2800
-Connection ~ 3950 2800
-Wire Wire Line
 	4100 2700 3250 2700
 Wire Wire Line
@@
 	3250 3200 4100 3200
 Wire Wire Line
-	3950 3300 4100 3300
-Connection ~ 3950 3300
-Wire Wire Line
 	3250 3500 4100 3500
 Wire Wire Line
@@
 	3250 3700 4100 3700
 Wire Wire Line
-	3950 3800 4100 3800
-Connection ~ 3950 3800
-Wire Wire Line
 	4100 3900 3250 3900
 Wire Wire Line
@@
 Wire Wire Line
 	3250 4200 4100 4200
-Wire Wire Line
-	4100 4300 3400 4300
-Connection ~ 3400 4300
 Wire Wire Line
 	3250 4400 4100 4400
@@
 	1850 3200 1200 3200
 Wire Wire Line
-	1200 3300 1750 3300
-Connection ~ 1750 3300
-Wire Wire Line
 	1850 3400 1200 3400
 Wire Wire Line
@@
 Wire Wire Line
 	1200 2700 1850 2700
-Wire Wire Line
-	1750 2800 1200 2800
-Connection ~ 1750 2800
 Wire Wire Line
 	1200 2900 1850 2900
@@
 Wire Wire Line
 	2650 2400 2650 2000
-Wire Wire Line
-	2550 2000 2550 2250
-Connection ~ 2550 2250
 Wire Wire Line
 	2450 2000 2450 2400
@@
 Wire Wire Line
 	1450 4400 1850 4400
+Wire Wire Line
+	1200 2800 1850 2800
+Wire Wire Line
+	1200 3300 1850 3300
+Wire Wire Line
+	3250 4300 4100 4300
+Wire Wire Line
+	3250 2800 4100 2800
+Wire Wire Line
+	3250 3300 4100 3300
+Wire Wire Line
+	3250 3800 4100 3800
+Wire Wire Line
+	2550 2000 2550 2400
 $EndSCHEMATC

Commit message: Correct wrong part names and PNs
Parts:
- R16, R17: PN CRCW080510K0FKEA -> CRCW080547K0FKEA
Changed lines of the file:
@@
 F 3 "~" H 8150 3800 50  0001 C CNN
 F 4 "Vishay" H 8150 3800 50  0001 C CNN "MFN"
-F 5 "CRCW080510K0FKEA" H 8150 3800 50  0001 C CNN "PN"
+F 5 "CRCW080547K0FKEA" H 8150 3800 50  0001 C CNN "PN"
 	1    8150 3800
 	1    0    0    -1
@@
 F 3 "~" H 8050 5150 50  0001 C CNN
 F 4 "Vishay" H 8050 5150 50  0001 C CNN "MFN"
-F 5 "CRCW080510K0FKEA" H 8050 5150 50  0001 C CNN "PN"
+F 5 "CRCW080547K0FKEA" H 8050 5150 50  0001 C CNN "PN"
 	1    8050 5150
 	1    0    0    -1

Commit message: Update non-available parts and add missing usb isolator to bom
Parts:
- added U6: adafruit_usb_isolator, adafruit:usb_isolator, symbol adafruit:adafruit_usb_isolator
- R10, R11: footprint Resistor_SMD:R_0603_1608Metric -> Resistor_SMD:R_1206_3216Metric; MFN Susumu -> Vishay; PN RR0816P-4990-D-68A -> CRCW1206510RJNEA
Connections:
- net labels removed: adafruit_usb_isolator
Changed lines of the file:
@@
 F 0 "R10" V 7543 3600 50  0000 C CNN
 F 1 "500" V 7634 3600 50  0000 C CNN
-F 2 "Resistor_SMD:R_0603_1608Metric" V 7680 3600 50  0001 C CNN
+F 2 "Resistor_SMD:R_1206_3216Metric" V 7680 3600 50  0001 C CNN
 F 3 "" H 7750 3600 50  0001 C CNN
-F 4 "Susumu" V 7750 3600 50  0001 C CNN "MFN"
-F 5 "RR0816P-4990-D-68A" V 7750 3600 50  0001 C CNN "PN"
+F 4 "Vishay" V 7750 3600 50  0001 C CNN "MFN"
+F 5 "CRCW1206510RJNEA" V 7750 3600 50  0001 C CNN "PN"
 	1    7750 3600
 	0    1    1    0
@@
 F 0 "R11" V 7443 4950 50  0000 C CNN
 F 1 "500" V 7534 4950 50  0000 C CNN
-F 2 "Resistor_SMD:R_0603_1608Metric" V 7580 4950 50  0001 C CNN
+F 2 "Resistor_SMD:R_1206_3216Metric" V 7580 4950 50  0001 C CNN
 F 3 "~" H 7650 4950 50  0001 C CNN
-F 4 "Susumu" H 7650 4950 50  0001 C CNN "MFN"
-F 5 "RR0816P-4990-D-68A" H 7650 4950 50  0001 C CNN "PN"
+F 4 "Vishay" H 7650 4950 50  0001 C CNN "MFN"
+F 5 "CRCW1206510RJNEA" H 7650 4950 50  0001 C CNN "PN"
 	1    7650 4950
 	0    1    1    0
@@
 	3450 1800 5650 1800
 $Comp
-L adafruit:adafruit_usb_isolator #Footprint1
+L adafruit:adafruit_usb_isolator U6
 U 1 1 616E0E33
 P 3300 6650
-F 0 "#Footprint1" H 3275 7155 50  0000 C CNN
+F 0 "U6" H 3275 7155 50  0000 C CNN
 F 1 "adafruit_usb_isolator" H 3275 7064 50  0000 C CNN
 F 2 "adafruit:usb_isolator" H 3275 6973 50  0000 C CNN
 F 3 "" H 3300 6650 50  0001 C CNN
+F 4 "Adafruit" H 3300 6650 50  0001 C CNN "MFN"
+F 5 "2107" H 3300 6650 50  0001 C CNN "PN"
 	1    3300 6650
 	1    0    0    -1

Commit message: Change 74LVC1G07GV to 74LVC1G17GV
The component 74LVC1G07GV is a drain-open-output device which would need a pull-up resistor to work as intended. Replace by Schmitt-Trigger 74LVC1G17GV.
Parts:
- U2: value 74LVC1G07 -> 74LVC1G17; PN 74LVC1G07GV -> 74LVC1G17GV
Changed lines of the file:
@@
 AR Path="/61464E7A/614769FF" Ref="U?"  Part="1"
 F 0 "U2" H 7394 3646 50  0000 L CNN
-F 1 "74LVC1G07" H 7394 3555 50  0000 L CNN
+F 1 "74LVC1G17" H 7394 3555 50  0000 L CNN
 F 2 "Package_TO_SOT_SMD:SOT-23-5" H 7700 3350 50  0001 C CNN
 F 3 "https://assets.nexperia.com/documents/data-sheet/74LVC1G07.pdf" H 6650 3400 50  0001 C CNN
 F 4 "Nexperia" H 7050 3600 50  0001 C CNN "MFN"
-F 5 "74LVC1G07GV" H 7050 3600 50  0001 C CNN "PN"
+F 5 "74LVC1G17GV" H 7050 3600 50  0001 C CNN "PN"
 	1    7050 3600
 	-1   0    0    -1
