File: KiCAD/output_buffer.sch (KiCad schematic (older format))
At the start: 7 parts, among them U2 74ABT245

Commit message: rearranged input buffer
Parts:
- renumbered C5 to C4, R14 to R6, R16 to R7, R18 to R8, R20 to R9, U2 to U4
Changed lines of the file:
@@
 $Descr A4 11693 8268
 encoding utf-8
-Sheet 4 6
+Sheet 4 4
 Title "Prawnblaster Breakout Board, Output Buffers"
 Date "2020-12-11"
@@
 $EndDescr
 $Comp
-L Device:R R18
+L Device:R R8
 U 1 1 5859C34F
 P 2150 2600
-F 0 "R18" V 2230 2600 50  0000 C CNN
+F 0 "R8" V 2230 2600 50  0000 C CNN
 F 1 "10k" V 2150 2600 50  0000 C CNN
 F 2 "Resistor_SMD:R_0805_2012Metric" V 2080 2600 50  0001 C CNN
@@
 $EndComp
 $Comp
-L Device:R R20
+L Device:R R9
 U 1 1 5859C356
 P 2350 2600
-F 0 "R20" V 2430 2600 50  0000 C CNN
+F 0 "R9" V 2430 2600 50  0000 C CNN
 F 1 "10k" V 2350 2600 50  0000 C CNN
 F 2 "Resistor_SMD:R_0805_2012Metric" V 2280 2600 50  0001 C CNN
@@
 $EndComp
 $Comp
-L Device:R R16
+L Device:R R7
 U 1 1 5859C35D
 P 1950 2600
-F 0 "R16" V 2030 2600 50  0000 C CNN
+F 0 "R7" V 2030 2600 50  0000 C CNN
 F 1 "10k" V 1950 2600 50  0000 C CNN
 F 2 "Resistor_SMD:R_0805_2012Metric" V 1880 2600 50  0001 C CNN
@@
 $EndComp
 $Comp
-L Device:R R14
+L Device:R R6
 U 1 1 5859C364
 P 1750 2600
-F 0 "R14" V 1830 2600 50  0000 C CNN
+F 0 "R6" V 1830 2600 50  0000 C CNN
 F 1 "10k" V 1750 2600 50  0000 C CNN
 F 2 "Resistor_SMD:R_0805_2012Metric" V 1680 2600 50  0001 C CNN
@@
 $EndComp
 $Comp
-L power:GND #PWR029
+L power:GND #PWR019
 U 1 1 5859C371
 P 3850 3100
-F 0 "#PWR029" H 3850 2850 50  0001 C CNN
+F 0 "#PWR019" H 3850 2850 50  0001 C CNN
 F 1 "GND" H 3850 2950 50  0000 C CNN
 F 2 "" H 3850 3100 50  0000 C CNN
@@
 $EndComp
 $Comp
-L power:GND #PWR031
+L power:GND #PWR020
 U 1 1 5859C455
 P 4150 1300
-F 0 "#PWR031" H 4150 1050 50  0001 C CNN
+F 0 "#PWR020" H 4150 1050 50  0001 C CNN
 F 1 "GND" H 4150 1150 50  0000 C CNN
 F 2 "" H 4150 1300 50  0000 C CNN
@@
 $EndComp
 $Comp
-L power:GND #PWR027
+L power:GND #PWR018
 U 1 1 5859C48A
 P 3200 2800
-F 0 "#PWR027" H 3200 2550 50  0001 C CNN
+F 0 "#PWR018" H 3200 2550 50  0001 C CNN
 F 1 "GND" H 3200 2650 50  0000 C CNN
 F 2 "" H 3200 2800 50  0000 C CNN
@@
 Vcc
 $Comp
-L Device:C C5
+L Device:C C4
 U 1 1 58595141
 P 4450 1100
-F 0 "C5" H 4475 1200 50  0000 L CNN
+F 0 "C4" H 4475 1200 50  0000 L CNN
 F 1 "10u" H 4475 1000 50  0000 L CNN
 F 2 "Capacitor_SMD:C_1210_3225Metric" H 4488 950 50  0001 C CNN
@@
 $EndComp
 $Comp
-L power:GND #PWR033
+L power:GND #PWR021
 U 1 1 585954C8
 P 4450 1300
-F 0 "#PWR033" H 4450 1050 50  0001 C CNN
+F 0 "#PWR021" H 4450 1050 50  0001 C CNN
 F 1 "GND" H 4450 1150 50  0000 C CNN
 F 2 "" H 4450 1300 50  0000 C CNN
@@
 	2350 2450 2350 1750
 $Comp
-L power:GND #PWR019
+L power:GND #PWR014
 U 1 1 585D49B4
 P 1750 2800
-F 0 "#PWR019" H 1750 2550 50  0001 C CNN
+F 0 "#PWR014" H 1750 2550 50  0001 C CNN
 F 1 "GND" H 1755 2627 50  0000 C CNN
 F 2 "" H 1750 2800 50  0000 C CNN
@@
 $EndComp
 $Comp
-L power:GND #PWR021
+L power:GND #PWR015
 U 1 1 585D4A67
 P 1950 2800
-F 0 "#PWR021" H 1950 2550 50  0001 C CNN
+F 0 "#PWR015" H 1950 2550 50  0001 C CNN
 F 1 "GND" H 1955 2627 50  0000 C CNN
 F 2 "" H 1950 2800 50  0000 C CNN
@@
 $EndComp
 $Comp
-L power:GND #PWR023
+L power:GND #PWR016
 U 1 1 585D4AC6
 P 2150 2800
-F 0 "#PWR023" H 2150 2550 50  0001 C CNN
+F 0 "#PWR016" H 2150 2550 50  0001 C CNN
 F 1 "GND" H 2155 2627 50  0000 C CNN
 F 2 "" H 2150 2800 50  0000 C CNN
@@
 $EndComp
 $Comp
-L power:GND #PWR025
+L power:GND #PWR017
 U 1 1 585D4B25
 P 2350 2800
-F 0 "#PWR025" H 2350 2550 50  0001 C CNN
+F 0 "#PWR017" H 2350 2550 50  0001 C CNN
 F 1 "GND" H 2355 2627 50  0000 C CNN
 F 2 "" H 2350 2800 50  0000 C CNN
@@
 	2350 1750 3300 1750
 $Comp
-L 74xx:74LS245 U2
+L 74xx:74LS245 U4
 U 1 1 5FE1B5DA
 P 3850 2250
-F 0 "U2" H 3950 3150 50  0000 C CNN
+F 0 "U4" H 3950 3150 50  0000 C CNN
 F 1 "74ABT245" H 3650 3150 50  0000 C CNN
 F 2 "Package_SO:SOIC-20W_7.5x12.8mm_P1.27mm" H 3850 2250 50  0001 C CNN

Commit message: Add USB-isolator plus extra power supply; move parts
Connections:
- net labels added: Vcc_5V
- net labels removed: Vcc
Changed lines of the file:
@@
 $EndComp
 Text HLabel 3850 750  1    60   UnSpc ~ 0
-Vcc
+Vcc_5V
 Text HLabel 1350 1750 0    60   Input ~ 0
 A0
@@
 B3
 Text HLabel 3200 2600 1    60   UnSpc ~ 0
-Vcc
+Vcc_5V
 $Comp
 L Device:C C4
