File: KiCAD/power_supply.sch (KiCad schematic (older format))
At the start: 5 parts, among them J14 Conn_01x03, U1 78L05

Commit message: rearranged input buffer
Parts:
- renumbered J14 to J6, U1 to U3
Changed lines of the file:
@@
 $Descr A4 11693 8268
 encoding utf-8
-Sheet 2 6
+Sheet 2 4
 Title "Prawnblaster Breakout Board, Output Buffers"
 Date "2020-12-11"
@@
 $EndDescr
 $Comp
-L Regulator_Linear:LM7805_TO220 U1
+L Regulator_Linear:LM7805_TO220 U3
 U 1 1 585983FB
 P 6250 3550
-F 0 "U1" H 6400 3300 50  0000 C CNN
+F 0 "U3" H 6400 3300 50  0000 C CNN
 F 1 "78L05" H 6250 3750 50  0000 C CNN
 F 2 "Package_TO_SOT_THT:TO-220-3_Horizontal_TabDown" H 6250 3550 50  0001 C CNN
@@
 $EndComp
 $Comp
-L power:GND #PWR016
+L power:GND #PWR011
 U 1 1 58598402
 P 6250 3900
-F 0 "#PWR016" H 6250 3650 50  0001 C CNN
+F 0 "#PWR011" H 6250 3650 50  0001 C CNN
 F 1 "GND" H 6250 3750 50  0000 C CNN
 F 2 "" H 6250 3900 50  0000 C CNN
@@
 $EndComp
 $Comp
-L power:GND #PWR017
+L power:GND #PWR012
 U 1 1 5859841A
 P 6850 3950
-F 0 "#PWR017" H 6850 3700 50  0001 C CNN
+F 0 "#PWR012" H 6850 3700 50  0001 C CNN
 F 1 "GND" H 6855 3777 50  0000 C CNN
 F 2 "" H 6850 3950 50  0000 C CNN
@@
 $EndComp
 $Comp
-L power:GND #PWR015
+L power:GND #PWR010
 U 1 1 5859862F
 P 5200 3950
-F 0 "#PWR015" H 5200 3700 50  0001 C CNN
+F 0 "#PWR010" H 5200 3700 50  0001 C CNN
 F 1 "GND" H 5205 3777 50  0000 C CNN
 F 2 "" H 5200 3950 50  0000 C CNN
@@
 Connection ~ 5200 3550
 $Comp
-L power:GND #PWR014
+L power:GND #PWR09
 U 1 1 585987D9
 P 1900 3350
-F 0 "#PWR014" H 1900 3100 50  0001 C CNN
+F 0 "#PWR09" H 1900 3100 50  0001 C CNN
 F 1 "GND" H 1900 3200 50  0000 C CNN
 F 2 "" H 1900 3350 50  0000 C CNN
@@
 	1550 3550 2400 3550
 $Comp
-L Connector_Generic:Conn_01x03 J14
+L Connector_Generic:Conn_01x03 J6
 U 1 1 5FD3FE88
 P 1350 3450
-F 0 "J14" H 1250 3100 50  0000 C CNN
+F 0 "J6" H 1250 3100 50  0000 C CNN
 F 1 "Conn_01x03" H 1250 3200 50  0000 C CNN
 F 2 "Connector:FanPinHeader_1x03_P2.54mm_Vertical" H 1350 3450 50  0001 C CNN

Commit message: Add GND connections, update authorship
Connections:
- wire segments 20 -> 19
Changed lines of the file:
@@
 encoding utf-8
 Sheet 2 4
-Title "Prawnblaster Breakout Board, Output Buffers"
+Title "Prawnblaster Breakout Board, Power Supply"
 Date "2020-12-11"
 Rev "v1.0"
 Comp "TU Darmstadt, Institut für Angewandte Physik, AG Birkl"
 Comment1 "Email: patrick.baus@physik.tu-darmstadt.de"
-Comment2 "Design by: Patrick Baus and Lars Pause"
+Comment2 "Design by: Patrick Baus"
 Comment3 ""
 Comment4 ""
@@
 Wire Wire Line
 	1700 3450 1700 3300
-Wire Wire Line
-	1700 3300 1900 3300
-Wire Wire Line
-	1900 3300 1900 3350
 $Comp
 L Device:D D1
@@
 Wire Wire Line
 	6850 3550 7600 3550
-$Comp
-L power:PWR_FLAG #FLG01
-U 1 1 6002ED13
-P 1900 3250
-F 0 "#FLG01" H 1900 3325 50  0001 C CNN
-F 1 "PWR_FLAG" H 1900 3450 50  0000 C CNN
-F 2 "" H 1900 3250 50  0001 C CNN
-F 3 "~" H 1900 3250 50  0001 C CNN
-	1    1900 3250
-	1    0    0    -1
-$EndComp
 Wire Wire Line
-	1900 3250 1900 3300
-Connection ~ 1900 3300
+	1900 3300 1900 3350
+Wire Wire Line
+	1700 3300 1900 3300
 $EndSCHEMATC

Commit message: Add 64Pin Case Power Supply, update PCB dimensions and SMA-Type
Note: Pi Pico footprint is missing!
Parts:
- removed J6: Conn_01x03, Connector:FanPinHeader_1x03_P2.54mm_Vertical, symbol Connector_Generic:Conn_01x03
- added J6: C64AC, Custom_footprints_project:Socket_DIN41612-CaseC1-AC-Male-64Pin-2rows, symbol Connector:C64AC
Connections:
- wire segments 19 -> 41
- no-connect marks 1 -> 0
Changed lines of the file:
@@
 L Regulator_Linear:LM7805_TO220 U3
 U 1 1 585983FB
-P 6250 3550
-F 0 "U3" H 6400 3300 50  0000 C CNN
-F 1 "78L05" H 6250 3750 50  0000 C CNN
-F 2 "Package_TO_SOT_THT:TO-220-3_Horizontal_TabDown" H 6250 3550 50  0001 C CNN
-F 3 "" H 6250 3550 50  0000 C CNN
-F 4 "Fairchild" H 6250 3550 60  0001 C CNN "MFN"
-F 5 "LM7805CT" H 6250 3550 50  0001 C CNN "PN"
-	1    6250 3550
+P 6300 1550
+F 0 "U3" H 6450 1300 50  0000 C CNN
+F 1 "78L05" H 6300 1750 50  0000 C CNN
+F 2 "Package_TO_SOT_THT:TO-220-3_Horizontal_TabDown" H 6300 1550 50  0001 C CNN
+F 3 "" H 6300 1550 50  0000 C CNN
+F 4 "Fairchild" H 6300 1550 60  0001 C CNN "MFN"
+F 5 "LM7805CT" H 6300 1550 50  0001 C CNN "PN"
+	1    6300 1550
 	1    0    0    -1
 $EndComp
@@
 L power:GND #PWR011
 U 1 1 58598402
-P 6250 3900
-F 0 "#PWR011" H 6250 3650 50  0001 C CNN
-F 1 "GND" H 6250 3750 50  0000 C CNN
-F 2 "" H 6250 3900 50  0000 C CNN
-F 3 "" H 6250 3900 50  0000 C CNN
-	1    6250 3900
-	1    0    0    -1
-$EndComp
-Connection ~ 6850 3550
-Wire Wire Line
-	6250 3850 6250 3900
+P 6300 1900
+F 0 "#PWR011" H 6300 1650 50  0001 C CNN
+F 1 "GND" H 6300 1750 50  0000 C CNN
+F 2 "" H 6300 1900 50  0000 C CNN
+F 3 "" H 6300 1900 50  0000 C CNN
+	1    6300 1900
+	1    0    0    -1
+$EndComp
+Connection ~ 6900 1550
+Wire Wire Line
+	6300 1850 6300 1900
 $Comp
 L Device:CP C2
 U 1 1 58598413
-P 6850 3750
-F 0 "C2" H 6968 3796 50  0000 L CNN
-F 1 "47u" H 6968 3705 50  0000 L CNN
-F 2 "Capacitor_THT:CP_Radial_D6.3mm_P2.50mm" H 6888 3600 50  0001 C CNN
-F 3 "" H 6850 3750 50  0000 C CNN
-F 4 "Panasonic" H 6850 3750 60  0001 C CNN "MFN"
-F 5 "EEUFR1J470" H 6850 3750 50  0001 C CNN "PN"
-	1    6850 3750
+P 6900 1750
+F 0 "C2" H 7018 1796 50  0000 L CNN
+F 1 "47u" H 7018 1705 50  0000 L CNN
+F 2 "Capacitor_THT:CP_Radial_D6.3mm_P2.50mm" H 6938 1600 50  0001 C CNN
+F 3 "" H 6900 1750 50  0000 C CNN
+F 4 "Panasonic" H 6900 1750 60  0001 C CNN "MFN"
+F 5 "EEUFR1J470" H 6900 1750 50  0001 C CNN "PN"
+	1    6900 1750
 	1    0    0    -1
 $EndComp
@@
 L power:GND #PWR012
 U 1 1 5859841A
-P 6850 3950
-F 0 "#PWR012" H 6850 3700 50  0001 C CNN
-F 1 "GND" H 6855 3777 50  0000 C CNN
-F 2 "" H 6850 3950 50  0000 C CNN
-F 3 "" H 6850 3950 50  0000 C CNN
-	1    6850 3950
-	1    0    0    -1
-$EndComp
-Wire Wire Line
-	6850 3900 6850 3950
-Wire Wire Line
-	6850 3200 6850 3550
-Wire Wire Line
-	4250 3550 5200 3550
-Connection ~ 5600 3550
-Wire Wire Line
-	5600 3200 5600 3550
+P 6900 1950
+F 0 "#PWR012" H 6900 1700 50  0001 C CNN
+F 1 "GND" H 6905 1777 50  0000 C CNN
+F 2 "" H 6900 1950 50  0000 C CNN
+F 3 "" H 6900 1950 50  0000 C CNN
+	1    6900 1950
+	1    0    0    -1
+$EndComp
+Wire Wire Line
+	6900 1900 6900 1950
+Wire Wire Line
+	6900 1200 6900 1550
+Wire Wire Line
+	4300 1550 5250 1550
+Connection ~ 5650 1550
+Wire Wire Line
+	5650 1200 5650 1550
 $Comp
 L Device:CP C1
 U 1 1 58598629
-P 5200 3750
-F 0 "C1" H 5318 3796 50  0000 L CNN
-F 1 "47u" H 5318 3705 50  0000 L CNN
-F 2 "Capacitor_THT:CP_Radial_D6.3mm_P2.50mm" H 5238 3600 50  0001 C CNN
-F 3 "" H 5200 3750 50  0000 C CNN
-F 4 "Panasonic" H 5200 3750 60  0001 C CNN "MFN"
-F 5 "EEUFR1J470" H 5200 3750 50  0001 C CNN "PN"
-	1    5200 3750
+P 5250 1750
+F 0 "C1" H 5368 1796 50  0000 L CNN
+F 1 "47u" H 5368 1705 50  0000 L CNN
+F 2 "Capacitor_THT:CP_Radial_D6.3mm_P2.50mm" H 5288 1600 50  0001 C CNN
+F 3 "" H 5250 1750 50  0000 C CNN
+F 4 "Panasonic" H 5250 1750 60  0001 C CNN "MFN"
+F 5 "EEUFR1J470" H 5250 1750 50  0001 C CNN "PN"
+	1    5250 1750
 	1    0    0    -1
 $EndComp
@@
 L power:GND #PWR010
 U 1 1 5859862F
-P 5200 3950
-F 0 "#PWR010" H 5200 3700 50  0001 C CNN
-F 1 "GND" H 5205 3777 50  0000 C CNN
-F 2 "" H 5200 3950 50  0000 C CNN
-F 3 "" H 5200 3950 50  0000 C CNN
-	1    5200 3950
-	1    0    0    -1
-$EndComp
-Wire Wire Line
-	5200 3900 5200 3950
-Wire Wire Line
-	5200 3600 5200 3550
-Connection ~ 5200 3550
+P 5250 1950
+F 0 "#PWR010" H 5250 1700 50  0001 C CNN
+F 1 "GND" H 5255 1777 50  0000 C CNN
+F 2 "" H 5250 1950 50  0000 C CNN
+F 3 "" H 5250 1950 50  0000 C CNN
+	1    5250 1950
+	1    0    0    -1
+$EndComp
+Wire Wire Line
+	5250 1900 5250 1950
+Wire Wire Line
+	5250 1600 5250 1550
+Connection ~ 5250 1550
 $Comp
 L power:GND #PWR09
 U 1 1 585987D9
-P 1900 3350
-F 0 "#PWR09" H 1900 3100 50  0001 C CNN
-F 1 "GND" H 1900 3200 50  0000 C CNN
-F 2 "" H 1900 3350 50  0000 C CNN
-F 3 "" H 1900 3350 50  0000 C CNN
-	1    1900 3350
-	1    0    0    -1
-$EndComp
-Wire Wire Line
-	1550 3450 1700 3450
-Wire Wire Line
-	1700 3450 1700 3300
+P 1350 4400
+F 0 "#PWR09" H 1350 4150 50  0001 C CNN
+F 1 "GND" H 1350 4250 50  0000 C CNN
+F 2 "" H 1350 4400 50  0000 C CNN
+F 3 "" H 1350 4400 50  0000 C CNN
+	1    1350 4400
+	1    0    0    -1
+$EndComp
 $Comp
 L Device:D D1
 U 1 1 58598927
-P 6250 3200
-F 0 "D1" H 6250 3415 50  0000 C CNN
-F 1 "D" H 6250 3324 50  0000 C CNN
-F 2 "Diode_SMD:D_SMB" H 6250 3200 50  0001 C CNN
-F 3 "" H 6250 3200 50  0000 C CNN
-F 4 "Vishay" H 6250 3200 60  0001 C CNN "MFN"
-F 5 "S2B-E3/52T" H 6250 3200 50  0001 C CNN "PN"
-	1    6250 3200
-	1    0    0    -1
-$EndComp
-Wire Wire Line
-	6400 3200 6850 3200
-Wire Wire Line
-	6100 3200 5600 3200
-Text Notes 6550 2950 0    60   ~ 0
+P 6300 1200
+F 0 "D1" H 6300 1415 50  0000 C CNN
+F 1 "D" H 6300 1324 50  0000 C CNN
+F 2 "Diode_SMD:D_SMB" H 6300 1200 50  0001 C CNN
+F 3 "" H 6300 1200 50  0000 C CNN
+F 4 "Vishay" H 6300 1200 60  0001 C CNN "MFN"
+F 5 "S2B-E3/52T" H 6300 1200 50  0001 C CNN "PN"
+	1    6300 1200
+	1    0    0    -1
+$EndComp
+Wire Wire Line
+	6450 1200 6900 1200
+Wire Wire Line
+	6150 1200 5650 1200
+Text Notes 6600 950  0    60   ~ 0
 Protection diode, because of the high output capacitance.\nCan be of any 1N4002 or higher type.
-Text HLabel 7600 3550 2    60   UnSpc ~ 0
+Text HLabel 7650 1550 2    60   UnSpc ~ 0
 Vcc
 $Sheet
-S 2400 3400 1850 500
+S 2450 1400 1850 500
 U 5859057F
 F0 "Reverse Polarity Protection" 60
 F1 "reverse_polarity_protection.sch" 60
-F2 "V18_unprot" U L 2400 3550 60
-F3 "V18" U R 4250 3550 60
+F2 "V18_unprot" U L 2450 1550 60
+F3 "V18" U R 4300 1550 60
 $EndSheet
 Wire Wire Line
-	6550 3550 6850 3550
-Wire Wire Line
-	6850 3550 6850 3600
-Wire Wire Line
-	5600 3550 5950 3550
-Wire Wire Line
-	5200 3550 5600 3550
-NoConn ~ 1550 3350
-Wire Wire Line
-	1550 3550 2400 3550
-$Comp
-L Connector_Generic:Conn_01x03 J6
-U 1 1 5FD3FE88
-P 1350 3450
-F 0 "J6" H 1250 3100 50  0000 C CNN
-F 1 "Conn_01x03" H 1250 3200 50  0000 C CNN
-F 2 "Connector:FanPinHeader_1x03_P2.54mm_Vertical" H 1350 3450 50  0001 C CNN
-F 3 "~" H 1350 3450 50  0001 C CNN
-F 4 "PSS 254/3G" H 1350 3450 50  0001 C CNN "PN"
-	1    1350 3450
-	-1   0    0    1
-$EndComp
-Wire Wire Line
-	6850 3550 7600 3550
-Wire Wire Line
-	1900 3300 1900 3350
-Wire Wire Line
-	1700 3300 1900 3300
+	6600 1550 6900 1550
+Wire Wire Line
+	6900 1550 6900 1600
+Wire Wire Line
+	5650 1550 6000 1550
+Wire Wire Line
+	5250 1550 5650 1550
+Wire Wire Line
+	2350 1550 2450 1550
+Wire Wire Line
+	6900 1550 7650 1550
+Wire Wire Line
+	1350 4350 1350 4400
+Wire Wire Line
+	1150 4350 1350 4350
+$Comp
+L Connector:C64AC J6
+U 1 1 614D9E5E
+P 750 4050
+F 0 "J6" H 668 7517 50  0000 C CNN
+F 1 "C64AC" H 668 7426 50  0000 C CNN
+F 2 "Custom_footprints_project:Socket_DIN41612-CaseC1-AC-Male-64Pin-2rows" H 750 4100 50  0001 C CNN
+F 3 " ~" H 750 4100 50  0001 C CNN
+	1    750  4050
+	-1   0    0    -1
+$EndComp
+Wire Wire Line
+	1050 3650 1150 3650
+Wire Wire Line
+	1150 3650 1150 3750
+Wire Wire Line
+	1150 4350 1050 4350
+Wire Wire Line
+	1050 4250 1150 4250
+Connection ~ 1150 4250
+Wire Wire Line
+	1150 4250 1150 4350
+Wire Wire Line
+	1050 4150 1150 4150
+Connection ~ 1150 4150
+Wire Wire Line
+	1150 4150 1150 4250
+Wire Wire Line
+	1050 4050 1150 4050
+Connection ~ 1150 4050
+Wire Wire Line
+	1150 4050 1150 4150
+Wire Wire Line
+	1050 3950 1150 3950
+Connection ~ 1150 3950
+Wire Wire Line
+	1150 3950 1150 4050
+Wire Wire Line
+	1050 3850 1150 3850
+Connection ~ 1150 3850
+Wire Wire Line
+	1150 3850 1150 3950
+Wire Wire Line
+	1050 3750 1150 3750
+Connection ~ 1150 3750
+Wire Wire Line
+	1150 3750 1150 3850
+Connection ~ 1150 4350
+Wire Wire Line
+	1050 850  1150 850
+Wire Wire Line
+	1150 850  1150 950
+Wire Wire Line
+	1150 1150 1050 1150
+Wire Wire Line
+	1050 1050 1150 1050
+Connection ~ 1150 1050
+Wire Wire Line
+	1150 1050 1150 1150
+Wire Wire Line
+	1050 950  1150 950
+Connection ~ 1150 950
+Wire Wire Line
+	1150 950  1150 1050
+Wire Wire Line
+	2350 1550 2350 1150
+Wire Wire Line
+	2350 1150 1150 1150
+Connection ~ 1150 1150
 $EndSCHEMATC

Commit message: Update MFN, PN and BOM
Parts:
- J6: MFN (none) -> Erni; PN (none) -> 364914
Changed lines of the file:
@@
 F 2 "Custom_footprints_project:Socket_DIN41612-CaseC1-AC-Male-64Pin-2rows" H 750 4100 50  0001 C CNN
 F 3 " ~" H 750 4100 50  0001 C CNN
+F 4 "Erni" H 750 4050 50  0001 C CNN "MFN"
+F 5 "364914" H 750 4050 50  0001 C CNN "PN"
 	1    750  4050
 	-1   0    0    -1

Commit message: Add USB-isolator plus extra power supply; move parts
Connections:
- net labels added: Vcc_5V
- net labels removed: Vcc
- no-connect marks 0 -> 52
Changed lines of the file:
@@
 Protection diode, because of the high output capacitance.\nCan be of any 1N4002 or higher type.
 Text HLabel 7650 1550 2    60   UnSpc ~ 0
-Vcc
+Vcc_5V
 $Sheet
 S 2450 1400 1850 500
@@
 	2350 1150 1150 1150
 Connection ~ 1150 1150
+NoConn ~ 1050 1250
+NoConn ~ 1050 1350
+NoConn ~ 1050 1450
+NoConn ~ 1050 1550
+NoConn ~ 1050 1650
+NoConn ~ 1050 1750
+NoConn ~ 1050 1850
+NoConn ~ 1050 1950
+NoConn ~ 1050 2050
+NoConn ~ 1050 2150
+NoConn ~ 1050 2250
+NoConn ~ 1050 2350
+NoConn ~ 1050 2450
+NoConn ~ 1050 2550
+NoConn ~ 1050 2650
+NoConn ~ 1050 2750
+NoConn ~ 1050 3550
+NoConn ~ 1050 3450
+NoConn ~ 1050 3350
+NoConn ~ 1050 3250
+NoConn ~ 1050 3150
+NoConn ~ 1050 3050
+NoConn ~ 1050 2950
+NoConn ~ 1050 2850
+NoConn ~ 1050 4450
+NoConn ~ 1050 4550
+NoConn ~ 1050 4650
+NoConn ~ 1050 4750
+NoConn ~ 1050 4850
+NoConn ~ 1050 4950
+NoConn ~ 1050 5050
+NoConn ~ 1050 5150
+NoConn ~ 1050 5250
+NoConn ~ 1050 5350
+NoConn ~ 1050 5450
+NoConn ~ 1050 5550
+NoConn ~ 1050 5650
+NoConn ~ 1050 5750
+NoConn ~ 1050 5850
+NoConn ~ 1050 5950
+NoConn ~ 1050 6050
+NoConn ~ 1050 6150
+NoConn ~ 1050 6250
+NoConn ~ 1050 6350
+NoConn ~ 1050 6450
+NoConn ~ 1050 6550
+NoConn ~ 1050 6650
+NoConn ~ 1050 6750
+NoConn ~ 1050 6850
+NoConn ~ 1050 6950
+NoConn ~ 1050 7050
+NoConn ~ 1050 7150
 $EndSCHEMATC

Commit message: Correct wrong part names and PNs
Parts:
- U3: value 78L05 -> 7805
Changed lines of the file:
@@
 P 6300 1550
 F 0 "U3" H 6450 1300 50  0000 C CNN
-F 1 "78L05" H 6300 1750 50  0000 C CNN
+F 1 "7805" H 6300 1750 50  0000 C CNN
 F 2 "Package_TO_SOT_THT:TO-220-3_Horizontal_TabDown" H 6300 1550 50  0001 C CNN
 F 3 "" H 6300 1550 50  0000 C CNN
