File: KiCAD/reverse_polarity_protection.sch (KiCad schematic (older format))
At the start: 3 parts, among them Q1 DMP6023LE

Commit message: rearranged input buffer
Parts:
- renumbered R13 to R5
Changed lines of the file:
@@
 $Descr A4 11693 8268
 encoding utf-8
-Sheet 3 6
+Sheet 3 4
 Title "Prawnblaster Breakout Board, Output Buffers"
 Date "2020-12-11"
@@
 	2350 2450 3650 2450
 $Comp
-L Device:R R13
+L Device:R R5
 U 1 1 57E2B631
 P 3950 3250
-F 0 "R13" V 4030 3250 50  0000 C CNN
+F 0 "R5" V 4030 3250 50  0000 C CNN
 F 1 "100k" V 3950 3250 50  0000 C CNN
 F 2 "Resistor_SMD:R_0805_2012Metric" V 3880 3250 50  0001 C CNN
@@
 $EndComp
 $Comp
-L power:GND #PWR018
+L power:GND #PWR013
 U 1 1 5800728F
 P 3950 3500
-F 0 "#PWR018" H 3950 3250 50  0001 C CNN
+F 0 "#PWR013" H 3950 3250 50  0001 C CNN
 F 1 "GND" H 3950 3350 50  0000 C CNN
 F 2 "" H 3950 3500 50  0000 C CNN

Commit message: Update MFN, PN and BOM
Parts:
- Q1: MFN (none) -> Diodes Incorporated
Changed lines of the file:
@@
 F 3 "" H 3950 2550 50  0000 C CNN
 F 4 "DMP6023LE-13" H 3950 2550 50  0001 C CNN "PN"
+F 5 "Diodes Incorporated" H 3950 2550 50  0001 C CNN "MFN"
 	1    3950 2550
 	0    -1   -1   0

Commit message: Update non-available parts and add missing usb isolator to bom
Other:
- note added: "Alternative:\nInfineon\nBSP613P H6327"
Changed lines of the file:
@@
 Wire Wire Line
 	5200 2450 5650 2450
+Text Notes 3300 2750 0    50   ~ 0
+Alternative:\nInfineon\nBSP613P H6327
 $EndSCHEMATC
